File: Platine/Studienarbeit.sch (KiCad schematic (older format))
At the start: 68 parts, among them J1 Conn_01x02_Female, J2 Conn_01x06_Female, J3 Conn_01x06_Female, J4 Conn_02x05_Odd_Even, J5 Conn_01x04_Female, J7 Conn_01x04_Female, Q1 IRF540NPBF, Q2 IRF540NPBF, Q3 IRF540NPBF, Q4 IRF540NPBF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

Commit message: To much to detect
Connections:
- wire segments 183 -> 184
Changed lines of the file:
@@
 Wire Wire Line
 	10900 6200 10800 6200
-$Comp
-L Connector:Conn_01x04_Female J5
-U 1 1 5ED67E70
-P 9150 6000
-F 0 "J5" H 9178 5976 50  0000 L CNN
-F 1 "Conn_01x04_Female" H 9178 5885 50  0000 L CNN
-F 2 "Connector_JST:JST_XH_B4B-XH-A_1x04_P2.50mm_Vertical" H 9150 6000 50  0001 C CNN
-F 3 "~" H 9150 6000 50  0001 C CNN
-	1    9150 6000
-	1    0    0    -1
-$EndComp
-Text Label 8950 6200 2    50   ~ 0
-MCR+
-Text Label 8950 6100 2    50   ~ 0
-MCR-
 Text Label 10000 2000 2    50   ~ 0
 MA2-
@@
 MA1-
 Text Label 9700 4300 2    50   ~ 0
-MA1+
+MA2+
 Text Label 9700 4700 2    50   ~ 0
-MA1-
+MA2-
 $Comp
 L Connector:Conn_01x04_Female J7
@@
 	1    0    0    -1
 $EndComp
+Text Label 4100 1550 3    50   Italic 0
+RESET
+Wire Wire Line
+	4100 1800 4100 1550
+Text Label 2550 6900 0    50   ~ 0
+VBAT
+Text Label 4100 2500 2    50   ~ 0
+C13
+Text Label 8950 6100 2    50   ~ 0
+MCR-
+$Comp
+L Connector:Conn_01x04_Female J5
+U 1 1 5ED67E70
+P 9150 6000
+F 0 "J5" H 9178 5976 50  0000 L CNN
+F 1 "Conn_01x04_Female" H 9178 5885 50  0000 L CNN
+F 2 "Connector_JST:JST_XH_B4B-XH-A_1x04_P2.50mm_Vertical" H 9150 6000 50  0001 C CNN
+F 3 "~" H 9150 6000 50  0001 C CNN
+	1    9150 6000
+	1    0    0    -1
+$EndComp
+Text Label 8950 6200 2    50   ~ 0
+MCR+
 $EndSCHEMATC

Commit message: platine final ready to order
Parts:
- removed J2, J3: Conn_01x06_Female, Connector_JST:JST_XH_B6B-XH-A_1x06_P2.50mm_Vertical, symbol Connector:Conn_01x06_Female
- removed J7: Conn_01x04_Female, Connector_JST:JST_XH_B4B-XH-A_1x04_P2.50mm_Vertical, symbol Connector:Conn_01x04_Female
- added J12, J7: 1755736, Studienarbeit:PhoenixContact1755736, symbol Studienarbeit:1755736
- added J13: Conn_01x02_Female, Connector_JST:JST_XH_B2B-XH-A_1x02_P2.50mm_Vertical, symbol Connector:Conn_01x02_Female
- added J14: Conn_01x02, Connector_PinHeader_2.54mm:PinHeader_1x02_P2.54mm_Vertical, symbol Connector_Generic:Conn_01x02
- 32.768: value Crystal -> Crystal 144-1100; footprint Crystal:Crystal_SMD_3215-2Pin_3.2x1.5mm -> Crystal:Crystal_SMD_2520-4Pin_2.5x2.0mm
- C1, C12, C13, C5, C9: LCSC (none) -> C136621
- C14, C15: value 0.1nF -> 100n; LCSC (none) -> C136621
- C18: footprint Capacitor_SMD:C_0805_2012Metric -> Capacitor_SMD:C_Elec_10x10.2
- C19: footprint Capacitor_SMD:C_0805_2012Metric -> Capacitor_SMD:C_Elec_8x6.2
- C2, C4: LCSC (none) -> C15850
- C3: value 10 nF -> 10 n
- D1, D2: LCSC (none) -> C2286
- D3: value 1N5824 -> MBRS540T3G; LCSC (none) -> C31849
- L1: footprint Inductor_SMD:L_0805_2012Metric -> Inductor_SMD:L_Wuerth_WE-PD-Typ-LS
- Opto: renamed from Opto2; LCSC (none) -> C146286
- Opto1, Opto3, Opto4, Opto5, Opto6: LCSC (none) -> C146286
- Q1, Q2, Q3, Q4, Q5, Q6: footprint Studienarbeit:IRF540NPBF -> Package_TO_SOT_THT:TO-220-3_Vertical
- R1, R8: LCSC (none) -> C17513
- R11, R16, R17, R19, R20, R3, R4, R5, R6, R7: LCSC (none) -> C17408
- R12: LCSC (none) -> C17437
- R18, R9: LCSC (none) -> C17414
- R2: LCDC (none) -> C17408
- U1: LCSC (none) -> C46243
- U2: LCSC (none) -> C8734
- U3: value LM4040DBZ-2.5 -> LM4040-2.5
- U4, U5: LCSC (none) -> C9932
- U6: LCSC (none) -> C12084
- U7: LCSC (none) -> C10002
Connections:
- net labels added: UART3_RX, UART3_TX
- net labels removed: A4, A5, VBAT
- wire segments 184 -> 188
