File: Platine/_autosave-Studienarbeit.sch (KiCad schematic (older format))
At the start: 68 parts, among them J1 Conn_01x02_Female, J2 Conn_01x06_Female, J3 Conn_01x06_Female, J4 Conn_02x05_Odd_Even, J5 Conn_01x04_Female, J7 Conn_01x04_Female, Q1 IRF540NPBF, Q2 IRF540NPBF, Q3 IRF540NPBF, Q4 IRF540NPBF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

Commit message: Platine
Connections:
- wire segments 183 -> 184
Changed lines of the file:
@@
 Wire Wire Line
 	10900 6200 10800 6200
-$Comp
-L Connector:Conn_01x04_Female J5
-U 1 1 5ED67E70
-P 9150 6000
-F 0 "J5" H 9178 5976 50  0000 L CNN
-F 1 "Conn_01x04_Female" H 9178 5885 50  0000 L CNN
-F 2 "Connector_JST:JST_XH_B4B-XH-A_1x04_P2.50mm_Vertical" H 9150 6000 50  0001 C CNN
-F 3 "~" H 9150 6000 50  0001 C CNN
-	1    9150 6000
-	1    0    0    -1
-$EndComp
-Text Label 8950 6200 2    50   ~ 0
-MCR+
-Text Label 8950 6100 2    50   ~ 0
-MCR-
 Text Label 10000 2000 2    50   ~ 0
 MA2-
@@
 	1    0    0    -1
 $EndComp
+Text Label 4100 1550 3    50   Italic 0
+RESET
+Wire Wire Line
+	4100 1800 4100 1550
+Text Label 2550 6900 0    50   ~ 0
+VBAT
+Text Label 4100 2500 2    50   ~ 0
+C13
+Text Label 8950 6100 2    50   ~ 0
+MCR-
+$Comp
+L Connector:Conn_01x04_Female J5
+U 1 1 5ED67E70
+P 9150 6000
+F 0 "J5" H 9178 5976 50  0000 L CNN
+F 1 "Conn_01x04_Female" H 9178 5885 50  0000 L CNN
+F 2 "Connector_JST:JST_XH_B4B-XH-A_1x04_P2.50mm_Vertical" H 9150 6000 50  0001 C CNN
+F 3 "~" H 9150 6000 50  0001 C CNN
+	1    9150 6000
+	1    0    0    -1
+$EndComp
+Text Label 8950 6200 2    50   ~ 0
+MCR+
 $EndSCHEMATC
