File: Platine/_autosave-Studienarbeit.sch (KiCad schematic (older format))
At the start: 69 parts, among them J1 Conn_01x02_Female, J12 1755736, J13 Conn_01x02_Female, J14 Conn_01x02, J4 Conn_02x05_Odd_Even, J5 Conn_01x04_Female, J7 1755736, Q1 IRF540NPBF, Q2 IRF540NPBF, Q3 IRF540NPBF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

Commit message: platine final ready to order
Parts:
- 32.768: footprint Crystal:Crystal_SMD_2520-4Pin_2.5x2.0mm -> Crystal:Crystal_SMD_2012-2Pin_2.0x1.2mm
- C1, C12, C13, C14, C15, C5, C9: LCSC (none) -> C136621
- C10, C11: LCSC (none) -> C1798
- C16, C17: LCSC (none) -> C46653
- C18: LCSC (none) -> C134782
- C19: LCSC (none) -> C127327
- C2, C4: LCSC (none) -> C15850
- C3: value 10 nF -> 10 n; LCSC (none) -> C1710
- D1, D2: LCSC (none) -> C2286
- D3: LCSC (none) -> C31849
- L1: LCSC (none) -> C169375
- Opto1, Opto2, Opto3, Opto4, Opto5, Opto6: LCSC (none) -> C146286
- R1, R8: LCSC (none) -> C17513
- R11, R16, R17, R19, R20, R3, R4, R5, R6, R7: LCSC (none) -> C17408
- R12: LCSC (none) -> C17437
- R18, R9: LCSC (none) -> C17414
- R2: LCDC (none) -> C17408
- U1: LCSC (none) -> C46243
- U2: LCSC (none) -> C8734
- U3: LCSC (none) -> C131939
- U4, U5: LCSC (none) -> C9932
- U6: LCSC (none) -> C12084
- U7: LCSC (none) -> C194349
