File: Platine/_autosave-Studienarbeit.kicad_pcb (KiCad board)
At the start: 2 copper layers, 85 x 100 mm, 100 parts, among them J1 Conn_01x02_Female, J10 1755736, J11 1755736, J12 1755736, J13 Conn_01x02_Female, J14 Conn_01x02, J2 1755736, J3 1755736, J4 Conn_02x05_Odd_Even, J5 Conn_01x04_Female, J6 Conn_01x04_Female, J7 1755736, J8 1755736, J9 1755736, Q1 IRF540NPBF, Q2 IRF540NPBF, Q3 IRF540NPBF, Q4 IRF540NPBF, Q5 IRF540NPBF, Q6 IRF540NPBF, SW1 SW_Push, U1 LD3985M33R_SOT23, U10 ADuM3190ARQZ, U11 RFM-0505S, U2 STM32F103C8Tx, U3 LM4040-2.5, U4 ACS712xLCTR-30A, U5 ACS712xLCTR-30A, U6 SN65HVD230, U7 LM2596S-5, U8 ADuM3190ARQZ, U9 RFM-0505S, Y1 8MHz

Commit message: platine final ready to order
Parts:
- 32.768: footprint Crystal:Crystal_SMD_2520-4Pin_2.5x2.0mm -> Crystal:Crystal_SMD_2012-2Pin_2.0x1.2mm
- C3: value 10 nF -> 10 n
- R21, R26: value 500 -> 470
- moved C3 37.1 mm to (169.2, 61.8), turned to 90 degrees
- moved C1 36.5 mm to (172.5, 60.5)
- moved U1 34.2 mm to (172.5, 63.8)
- moved C2 33.7 mm to (172.4, 58.2)
- moved C5 31.8 mm to (176.5, 65.5)
- moved C4 30.1 mm to (178.8, 65.5)
- moved C10 0.43 mm to (163.6, 98.2)
- moved C11 0.40 mm to (163.6, 94.3)
- moved R20 0.31 mm to (174.8, 79.7)
- turned C21 to 180 degrees
Routing:
- net +3V3: track 204.8 -> 117.3 mm, vias 5 -> 8
- net /A0: track 59.5 -> 32.2 mm, vias 0 -> 2
- net /A1: track 52.6 -> 27.2 mm, vias 0 -> 2
- net /CAN_TX: track 60.1 -> 42.0 mm, vias 0 -> 2
- net Net-(C21-Pad1): track 30.3 -> 15.2 mm
- net /PB2: track 35.6 -> 21.9 mm, vias 0 -> 2
- net /Sheet5EE7EB52/-IN1: track 32.9 -> 20.7 mm, vias 0 -> 2
- net GND: track 39.0 -> 27.4 mm, vias 83 -> 85
- net Net-(R11-Pad2): track 21.0 -> 11.5 mm
- net +5V: track 216.2 -> 208.9 mm, vias 9 -> 10
- net Net-(32.768-Pad1): track 18.9 -> 12.3 mm
- net /SWDIO: track 22.3 -> 15.7 mm, vias 0 -> 2
- net /PB1: track 25.0 -> 18.7 mm
- net /PB0: track 33.6 -> 28.4 mm, vias 0 -> 2
- net UART3_TX: track 38.2 -> 35.4 mm
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