File: Platine/file5EE7EB52.sch (KiCad schematic (older format))
At the start: 25 parts, among them J6 Conn_01x04_Female, U10 ADuM3190ARQZ, U11 RFM-0505S, U8 ADuM3190ARQZ, U9 RFM-0505S

Commit message: platine final ready to order
Parts:
- C20, C25: LCSC (none) -> C5378
- C21, C22, C23, C24, C26, C27, C28, C29: LCSC (none) -> C28323
- R13, R23: LCSC (none) -> C17633
- R14, R24: LCSC (none) -> C17513
- R15, R25: LCSC (none) -> C17604
- R21, R26: value 500 -> 470; LCSC (none) -> C17710
- R22, R27: LCSC (none) -> C17661
Connections:
- net GND: no longer C21.1, C22.1, U8.2 (GND1)
- new net: C21.1, C22.1, U8.2 (GND1)
Changed lines of the file:
@@
 $Descr A4 11693 8268
 encoding utf-8
-Sheet 2 2
+Sheet 2 3
 Title ""
 Date ""
@@
 F 2 "Resistor_SMD:R_0805_2012Metric" V 1430 3600 50  0001 C CNN
 F 3 "~" H 1500 3600 50  0001 C CNN
+F 4 " C17661" V 1500 3600 50  0001 C CNN "LCSC"
 	1    1500 3600
 	0    1    1    0
@@
 F 2 "Resistor_SMD:R_0805_2012Metric" V 980 3750 50  0001 C CNN
 F 3 "~" H 1050 3750 50  0001 C CNN
+F 4 "C17513" H 1050 3750 50  0001 C CNN "LCSC"
 	1    1050 3750
 	1    0    0    -1
@@
 F 2 "Resistor_SMD:R_0805_2012Metric" V 980 3450 50  0001 C CNN
 F 3 "~" H 1050 3450 50  0001 C CNN
+F 4 " C17633" H 1050 3450 50  0001 C CNN "LCSC"
 	1    1050 3450
 	1    0    0    -1
@@
 Wire Wire Line
 	1650 3600 2400 3600
-Text Label 2400 3800 2    50   ~ 0
-A2
 $Comp
 L Device:R R15
@@
 F 2 "Resistor_SMD:R_0805_2012Metric" V 1030 5250 50  0001 C CNN
 F 3 "~" H 1100 5250 50  0001 C CNN
+F 4 " C17604" H 1100 5250 50  0001 C CNN "LCSC"
 	1    1100 5250
 	1    0    0    -1
@@
 P 1300 4950
 F 0 "R21" V 1093 4950 50  0000 C CNN
-F 1 "500" V 1184 4950 50  0000 C CNN
+F 1 "470" V 1184 4950 50  0000 C CNN
 F 2 "Resistor_SMD:R_0805_2012Metric" V 1230 4950 50  0001 C CNN
 F 3 "~" H 1300 4950 50  0001 C CNN
+F 4 " C17710" V 1300 4950 50  0001 C CNN "LCSC"
 	1    1300 4950
 	0    1    1    0
@@
 F 2 "Capacitor_SMD:C_0805_2012Metric" H 1338 4450 50  0001 C CNN
 F 3 "~" H 1300 4600 50  0001 C CNN
+F 4 " C5378" V 1300 4600 50  0001 C CNN "LCSC"
 	1    1300 4600
 	0    1    1    0
@@
 Wire Wire Line
 	1450 4750 1450 4950
-Text Label 2400 3500 2    50   ~ 0
--IN1
 Wire Wire Line
 	1900 3300 1900 4050
@@
 F 2 "Resistor_SMD:R_0805_2012Metric" V 6780 3600 50  0001 C CNN
 F 3 "~" H 6850 3600 50  0001 C CNN
+F 4 " C17661" V 6850 3600 50  0001 C CNN "LCSC"
 	1    6850 3600
 	0    1    1    0
@@
 F 2 "Resistor_SMD:R_0805_2012Metric" V 6330 3750 50  0001 C CNN
 F 3 "~" H 6400 3750 50  0001 C CNN
+F 4 "C17513" H 6400 3750 50  0001 C CNN "LCSC"
 	1    6400 3750
 	1    0    0    -1
@@
 F 2 "Resistor_SMD:R_0805_2012Metric" V 6330 3450 50  0001 C CNN
 F 3 "~" H 6400 3450 50  0001 C CNN
+F 4 " C17633" H 6400 3450 50  0001 C CNN "LCSC"
 	1    6400 3450
 	1    0    0    -1
@@
 F 2 "Resistor_SMD:R_0805_2012Metric" V 6380 5250 50  0001 C CNN
 F 3 "~" H 6450 5250 50  0001 C CNN
+F 4 " C17604" H 6450 5250 50  0001 C CNN "LCSC"
 	1    6450 5250
 	1    0    0    -1
@@
 P 6650 4950
 F 0 "R26" V 6443 4950 50  0000 C CNN
-F 1 "500" V 6534 4950 50  0000 C CNN
+F 1 "470" V 6534 4950 50  0000 C CNN
 F 2 "Resistor_SMD:R_0805_2012Metric" V 6580 4950 50  0001 C CNN
 F 3 "~" H 6650 4950 50  0001 C CNN
+F 4 " C17710" V 6650 4950 50  0001 C CNN "LCSC"
 	1    6650 4950
-	0    1    1    0
-$EndComp
-$Comp
-L Device:C C25
-U 1 1 5EEBCE8D
-P 6650 4600
-F 0 "C25" V 6398 4600 50  0000 C CNN
-F 1 "220n" V 6489 4600 50  0000 C CNN
-F 2 "Capacitor_SMD:C_0805_2012Metric" H 6688 4450 50  0001 C CNN
-F 3 "~" H 6650 4600 50  0001 C CNN
-	1    6650 4600
 	0    1    1    0
 $EndComp
@@
 Wire Wire Line
 	9750 1300 10450 1300
-Wire Wire Line
-	2400 4200 2400 4300
-$Comp
-L Studienarbeit:ADuM3190ARQZ U8
-U 1 1 5EF0B225
-P 2400 2900
-F 0 "U8" H 3400 3287 60  0000 C CNN
-F 1 "ADuM3190ARQZ" H 3400 3181 60  0000 C CNN
-F 2 "Studienarbeit:ADuM3190ARQZ" H 3400 3140 60  0001 C CNN
-F 3 "" H 2400 2900 60  0000 C CNN
-	1    2400 2900
-	1    0    0    -1
-$EndComp
 $Comp
 L power:+5V #PWR?
@@
 $EndComp
 $Comp
-L Device:C C23
-U 1 1 5F0428BC
-P 4550 2900
-F 0 "C23" V 4802 2900 50  0000 C CNN
-F 1 "1u" V 4711 2900 50  0000 C CNN
-F 2 "Capacitor_SMD:C_0805_2012Metric" H 4588 2750 50  0001 C CNN
-F 3 "~" H 4550 2900 50  0001 C CNN
-	1    4550 2900
-	0    -1   -1   0
-$EndComp
-$Comp
 L Device:C C24
 U 1 1 5F044B92
@@
 F 2 "Capacitor_SMD:C_0805_2012Metric" H 4588 2950 50  0001 C CNN
 F 3 "~" H 4550 3100 50  0001 C CNN
+F 4 " C28323" V 4550 3100 50  0001 C CNN "LCSC"
 	1    4550 3100
 	0    -1   -1   0
 $EndComp
-Connection ~ 4400 2900
 $Comp
 L Device:C C21
@@
 F 2 "Capacitor_SMD:C_0805_2012Metric" H 2338 2750 50  0001 C CNN
 F 3 "~" H 2300 2900 50  0001 C CNN
+F 4 " C28323" V 2300 2900 50  0001 C CNN "LCSC"
 	1    2300 2900
 	0    -1   -1   0
@@
 F 2 "Capacitor_SMD:C_0805_2012Metric" H 2338 2950 50  0001 C CNN
 F 3 "~" H 2300 3100 50  0001 C CNN
+F 4 " C28323" V 2300 3100 50  0001 C CNN "LCSC"
 	1    2300 3100
 	0    -1   -1   0
 $EndComp
-Wire Wire Line
-	5100 4000 4400 4000
 Wire Wire Line
 	4700 2900 5100 2900
@@
 Wire Wire Line
 	2150 4200 2400 4200
-Connection ~ 2400 4200
 Wire Wire Line
 	2150 2900 2050 2900
@@
 	1    0    0    -1
 $EndComp
-Text Label 7750 3800 2    50   ~ 0
-A3
 Text Label 7750 3500 2    50   ~ 0
 -IN2
@@
 F 2 "Capacitor_SMD:C_0805_2012Metric" H 9938 2750 50  0001 C CNN
 F 3 "~" H 9900 2900 50  0001 C CNN
+F 4 " C28323" V 9900 2900 50  0001 C CNN "LCSC"
 	1    9900 2900
 	0    -1   -1   0
@@
 F 2 "Capacitor_SMD:C_0805_2012Metric" H 9938 2950 50  0001 C CNN
 F 3 "~" H 9900 3100 50  0001 C CNN
+F 4 " C28323" V 9900 3100 50  0001 C CNN "LCSC"
 	1    9900 3100
 	0    -1   -1   0
@@
 F 2 "Capacitor_SMD:C_0805_2012Metric" H 7688 2750 50  0001 C CNN
 F 3 "~" H 7650 2900 50  0001 C CNN
+F 4 " C28323" V 7650 2900 50  0001 C CNN "LCSC"
 	1    7650 2900
 	0    -1   -1   0
@@
 F 2 "Capacitor_SMD:C_0805_2012Metric" H 7688 2950 50  0001 C CNN
 F 3 "~" H 7650 3100 50  0001 C CNN
+F 4 " C28323" V 7650 3100 50  0001 C CNN "LCSC"
 	1    7650 3100
 	0    -1   -1   0
@@
 Wire Wire Line
 	9750 4000 9750 4100
-Connection ~ 2400 4300
+Wire Wire Line
+	2450 3100 2400 3100
+Wire Wire Line
+	2450 2900 2400 2900
+Text GLabel 7750 3800 0    50   Input ~ 0
+A3
+Text Label 2400 3500 2    50   ~ 0
+-IN1
 Wire Wire Line
 	2400 4300 2400 4400
 Connection ~ 4400 4000
-Wire Wire Line
-	2450 3100 2400 3100
-Wire Wire Line
-	2450 2900 2400 2900
 Connection ~ 2400 2900
+Wire Wire Line
+	5100 4000 4400 4000
+$Comp
+L Studienarbeit:ADuM3190ARQZ U8
+U 1 1 5EF0B225
+P 2400 2900
+F 0 "U8" H 3400 3287 60  0000 C CNN
+F 1 "ADuM3190ARQZ" H 3400 3181 60  0000 C CNN
+F 2 "Studienarbeit:ADuM3190ARQZ" H 3400 3140 60  0001 C CNN
+F 3 "" H 2400 2900 60  0000 C CNN
+	1    2400 2900
+	1    0    0    -1
+$EndComp
+Text GLabel 2400 3800 0    50   Input ~ 0
+A2
+Connection ~ 4400 2900
+$Comp
+L Device:C C23
+U 1 1 5F0428BC
+P 4550 2900
+F 0 "C23" V 4802 2900 50  0000 C CNN
+F 1 "1u" V 4711 2900 50  0000 C CNN
+F 2 "Capacitor_SMD:C_0805_2012Metric" H 4588 2750 50  0001 C CNN
+F 3 "~" H 4550 2900 50  0001 C CNN
+F 4 " C28323" V 4550 2900 50  0001 C CNN "LCSC"
+	1    4550 2900
+	0    -1   -1   0
+$EndComp
+$Comp
+L Device:C C25
+U 1 1 5EEBCE8D
+P 6650 4600
+F 0 "C25" V 6398 4600 50  0000 C CNN
+F 1 "220n" V 6489 4600 50  0000 C CNN
+F 2 "Capacitor_SMD:C_0805_2012Metric" H 6688 4450 50  0001 C CNN
+F 3 "~" H 6650 4600 50  0001 C CNN
+F 4 " C5378" V 6650 4600 50  0001 C CNN "LCSC"
+	1    6650 4600
+	0    1    1    0
+$EndComp
 $EndSCHEMATC
