File: Platine/Studienarbeit.kicad_pcb (KiCad board)
At the start: 2 copper layers, 140.2 x 100.7 mm, 93 parts, among them J1 Conn_01x02_Female, J2 Conn_01x06_Female, J3 Conn_01x06_Female, J4 Conn_02x05_Odd_Even, J5 Conn_01x04_Female, J6 Conn_01x04_Female, J7 Conn_01x04_Female, Q1 IRF540NPBF, Q2 IRF540NPBF, Q3 IRF540NPBF, Q4 IRF540NPBF, Q5 IRF540NPBF, Q6 IRF540NPBF, SW1 SW_Push, U1 LD3985M33R_SOT23, U10 ADuM3190ARQZ, U11 RFM-0505S, U2 STM32F103C8Tx, U3 LM4040DBZ-2.5, U4 ACS712xLCTR-30A, U5 ACS712xLCTR-30A, U6 SN65HVD230, U7 LM2596S-5, U8 ADuM3190ARQZ, U9 RFM-0505S, Y1 8MHz

Commit message: To much to detect
Parts:
- moved C14 329.5 mm to (171.8, 76.5), turned to 180 degrees
- moved U4 319.8 mm to (165.8, 72.2)
- moved D1 308.2 mm to (188.3, 69.1), turned to 270 degrees
- moved R1 300.4 mm to (190.2, 69.2), turned to 270 degrees
- moved R19 290.3 mm to (170.7, 77.9)
- moved C16 279.3 mm to (171.6, 73.8), turned to 90 degrees
- moved C17 276.9 mm to (171.5, 80.1), turned to 90 degrees
- moved C15 276.3 mm to (165.7, 68.0), turned to 180 degrees
- moved R17 272.9 mm to (173.6, 72.9), turned to 270 degrees
- moved R20 251.9 mm to (173.3, 79.0), turned to 270 degrees
- moved R16 251.2 mm to (170.7, 71.6)
- moved J7 224.6 mm to (158.8, 71.6), turned to 270 degrees
- moved U5 164.1 mm to (166.0, 78.5)
- moved U10 132.8 mm to (186.2, 114.6), turned to 180 degrees
- moved J6 122.6 mm to (158.0, 95.1), turned to 270 degrees
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Connections:
- U5 pad 1: /MA1+ -> /MA2+
- U5 pad 2: /MA1+ -> /MA2+
- U5 pad 3: /MA1- -> /MA2-
- U5 pad 4: /MA1- -> /MA2-
Routing:
- net +5V: track 39.0 -> 202.6 mm, vias 0 -> 5
- net +3V3: track 79.4 -> 149.9 mm, vias 0 -> 4
- net /A0: track 0.00 -> 56.9 mm
- net /A1: track 0.00 -> 51.3 mm
- net /CAN_TX: track 0.00 -> 49.7 mm
- net /Sheet5EE7EB52/MV2-: track 0.00 -> 44.4 mm, vias 0 -> 2
- net /Sheet5EE7EB52/-IN2: track 0.00 -> 38.1 mm
- net /MM2+: track 36.7 -> 74.5 mm
- net /MM3+: track 27.7 -> 63.9 mm
- net /PB5: track 0.00 -> 35.6 mm
- net /MM1+: track 48.3 -> 12.9 mm
- net /CAN_RX: track 0.00 -> 34.4 mm, vias 0 -> 2
- net /Sheet5EE7EB52/MV2+: track 0.00 -> 33.2 mm
- net /Sheet5EE7EB52/MV1-: track 0.00 -> 32.6 mm, vias 0 -> 4
- net (no net): track 0.00 -> 32.1 mm
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- added copper zone on F.Cu, net GND
Other:
- board size 140.2 x 100.7 mm -> 62 x 100 mm
- rule trace_min: 0.2 -> 0.25

Commit message: Platine fertig geroutet
ToDO:
5mm Leiterbahnbreite anpassen
GND Verbindungen vollständig herstellen
Kondensatoren prüfen SMD!!
Parts:
- R1, R10, R11, R12, R13, R14, R15, R16, R17, R18, R19, R2, R20, R21, R22, R23, R24, R25, R26, R27, R3, R4, R5, R6, R7, R8, R9: footprint Resistor_SMD:R_0201_0603Metric -> Resistor_SMD:R_0805_2012Metric
- moved R24 5.00 mm to (176.3, 112.6)
- moved R3 4.98 mm to (193.8, 105.2)
- moved R23 4.95 mm to (178.5, 108.5)
- moved R5 3.54 mm to (196.5, 82.1)
- moved D2 3.31 mm to (177.1, 83.5)
- moved R1 3.24 mm to (189.7, 66.0), turned to 90 degrees
- moved R12 2.64 mm to (163.7, 60.2), turned to 90 degrees
- moved U3 2.29 mm to (175.4, 103.6)
- moved R16 2.19 mm to (171.4, 69.5)
- moved R8 2.17 mm to (176.9, 87.1)
- moved R27 1.89 mm to (179.7, 114.4)
- moved U6 1.83 mm to (167.6, 60.1)
- moved R21 1.75 mm to (170.7, 122.2)
- moved R14 1.71 mm to (156.1, 115.1), turned to 180 degrees
- moved R13 1.55 mm to (157.1, 109.8)
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Routing:
- net /MCH: track 17.2 -> 26.6 mm
- net /PB1: track 24.9 -> 18.5 mm
- net Net-(Opto2-Pad1): track 1.96 -> 8.00 mm
- net Net-(R23-Pad2): track 2.84 -> 8.73 mm
- net /MCL: track 20.6 -> 25.1 mm
- net /PB3: track 14.5 -> 18.5 mm
- net /Sheet5EE7EB52/MV2+: track 33.2 -> 29.6 mm
- net /MCR-: track 2.05 -> 5.52 mm
- net /RESET: track 23.6 -> 26.6 mm
- net /A1: track 51.3 -> 48.4 mm
- net /A0: track 56.9 -> 59.5 mm
- net Net-(R11-Pad2): track 11.5 -> 14.0 mm
- net /Sheet5EE7EB52/MV1+: track 18.9 -> 16.5 mm
- net Net-(R18-Pad2): track 1.97 -> 4.10 mm
- net Net-(R13-Pad2): track 2.35 -> 4.46 mm
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- added copper zone on B.Cu, net GND
Other:
- net class Strom added: clearance 0.2, trace_width 5, via_dia 0.8, via_drill 0.4

Commit message: platine final ready to order
Parts:
- added J10: 1755736, Studienarbeit:PhoenixContact1755736, F.Cu at (223.0, 73.5)
- added J11: 1755736, Studienarbeit:PhoenixContact1755736, F.Cu at (223.0, 43.5)
- added J12: 1755736, Studienarbeit:PhoenixContact1755736, F.Cu at (155.8, 83.2)
- added J13: Conn_01x02_Female, Connector_JST:JST_XH_B2B-XH-A_1x02_P2.50mm_Vertical, F.Cu at (197.2, 128.0)
- added J14: Conn_01x02, Connector_PinHeader_2.54mm:PinHeader_1x02_P2.54mm_Vertical, F.Cu at (200.8, 81.5)
- added J8: 1755736, Studienarbeit:PhoenixContact1755736, F.Cu at (223.0, 88.5)
- added J9: 1755736, Studienarbeit:PhoenixContact1755736, F.Cu at (223.0, 58.5)
- 32.768: value Crystal -> Crystal 144-1100; footprint Crystal:Crystal_SMD_3215-2Pin_3.2x1.5mm -> Crystal:Crystal_SMD_2012-2Pin_2.0x1.2mm
- C14, C15: value 0.1nF -> 100n
- C18: footprint Capacitor_SMD:C_0805_2012Metric -> Capacitor_SMD:C_Elec_10x10.2
- C19: footprint Capacitor_SMD:C_0805_2012Metric -> Capacitor_SMD:C_Elec_8x6.2
- C3: value 10 nF -> 10 n
- D3: value 1N5824 -> MBRS540T3G
- J2, J3: value Conn_01x06_Female -> 1755736; footprint Connector_JST:JST_XH_B6B-XH-A_1x06_P2.50mm_Vertical -> Studienarbeit:PhoenixContact1755736
- J7: value Conn_01x04_Female -> 1755736; footprint Connector_JST:JST_XH_B4B-XH-A_1x04_P2.50mm_Vertical -> Studienarbeit:PhoenixContact1755736
- L1: footprint Inductor_SMD:L_0805_2012Metric -> Inductor_SMD:L_Wuerth_WE-PD-Typ-LS
- Q1, Q2, Q3, Q4, Q5, Q6: footprint Studienarbeit:IRF540NPBF -> Package_TO_SOT_THT:TO-220-3_Vertical
- R21, R26: value 500 -> 470
- U3: value LM4040DBZ-2.5 -> LM4040-2.5
- moved J2 73.3 mm to (223.0, 118.5), turned to 270 degrees
- moved J3 56.6 mm to (223.0, 103.5), turned to 270 degrees
- moved C18 36.7 mm to (159.5, 41.0), turned to 180 degrees
- moved C3 36.3 mm to (169.2, 61.8), turned to 90 degrees
- moved U1 32.8 mm to (172.5, 63.8), turned to 180 degrees
- moved C5 30.5 mm to (176.5, 65.5)
- moved C4 28.8 mm to (178.8, 65.5)
- moved C1 28.1 mm to (172.5, 60.5)
- moved C2 25.1 mm to (172.4, 58.2)
- moved Q6 21.0 mm to (213.0, 43.5)
- moved Q5 17.9 mm to (213.0, 58.5)
- moved Q4 14.5 mm to (213.0, 73.5)
- moved L1 13.9 mm to (196.0, 47.5), turned to 270 degrees
- moved Opto5 13.4 mm to (207.2, 63.0), turned to 0 degrees
- moved Opto6 12.3 mm to (206.8, 51.8), turned to 0 degrees
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Connections:
- net /A4 renamed Net-(U2-Pad14)
- net /A5 renamed Net-(U2-Pad15)
- net /MM1+ renamed MM1+
- net /MM2- renamed MM2-
- C21 pad 1: GND -> Net-(C21-Pad1)
- C22 pad 1: GND -> Net-(C21-Pad1)
- J2 pad 2: /MM2+ -> MM1-
- J3 pad 1: /MM1- -> MM2+
- Opto1 pad 3: /MM1- -> MM1-
- Opto3 pad 3: /MM3- -> MM3-
- Opto4 pad 3: /MM4- -> MM4-
- Opto5 pad 3: /MM5- -> MM5-
- Opto6 pad 3: /MM6- -> MM6-
- Q1 pad 3: /MM1- -> MM1-
- Q2 pad 2: /MM2+ -> MM2+
- Q3 pad 2: /MM3+ -> MM3+
- Q3 pad 3: /MM3- -> MM3-
- Q4 pad 2: /MM4+ -> MM4+
- Q4 pad 3: /MM4- -> MM4-
- Q5 pad 2: /MM5+ -> MM5+
- Q5 pad 3: /MM5- -> MM5-
- Q6 pad 2: /MM6+ -> MM6+
- Q6 pad 3: /MM6- -> MM6-
- U10 pad 7: /Sheet5EE7EB52/A3 -> A3
- U2 pad 1: +3V3 -> Net-(J14-Pad2)
- U2 pad 12: /A2 -> A2
- U2 pad 13: /A3 -> A3
- U2 pad 21: Net-(U2-Pad21) -> UART3_TX
- U2 pad 22: Net-(U2-Pad22) -> UART3_RX
- U7 pad 4: Net-(U7-Pad4) -> +5V
- U8 pad 2: GND -> Net-(C21-Pad1)
- U8 pad 7: /Sheet5EE7EB52/A2 -> A2
Routing:
- net /MM1-: track 86.3 -> 0.00 mm
- net MM2-: track 79.8 -> 4.76 mm, vias 2 -> 0
- net /MM2+: track 74.5 -> 0.00 mm
- net /MM3-: track 68.5 -> 0.00 mm, vias 2 -> 0
- net /MM4-: track 65.3 -> 0.00 mm, vias 2 -> 0
- net /MM3+: track 63.9 -> 0.00 mm
- net /MM5-: track 57.8 -> 0.00 mm, vias 2 -> 0
- net /MM4+: track 54.5 -> 0.00 mm
- net /MM6-: track 48.7 -> 0.00 mm, vias 2 -> 0
- net /MM5+: track 45.4 -> 0.00 mm
- net UART3_RX: track 0.00 -> 36.4 mm, vias 0 -> 2
- net /MM6+: track 36.0 -> 0.00 mm
- net UART3_TX: track 0.00 -> 35.4 mm, vias 0 -> 2
- net (no net): track 32.1 -> 0.00 mm
- net Net-(J14-Pad2): track 0.00 -> 31.2 mm, vias 0 -> 2
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- added copper zone on F.Cu, net /MA1+
- added copper zone on F.Cu, net /MA1-
- added copper zone on F.Cu, net /MA2+
- added copper zone on F.Cu, net /MA2-
- added copper zone on F.Cu, net MM1+
- added copper zone on F.Cu, net MM1-
- added copper zone on F.Cu, net MM2+
- added copper zone on F.Cu, net MM2-
- added copper zone on F.Cu, net MM3+
- added copper zone on F.Cu, net MM3-
- added copper zone on F.Cu, net MM4+
- added copper zone on F.Cu, net MM4-
- added copper zone on F.Cu, net MM5+
- added copper zone on F.Cu, net MM5-
- added copper zone on F.Cu, net MM6+
- added copper zone on F.Cu, net MM6-
Other:
- board size 62 x 100 mm -> 85 x 100 mm
- net class Amperemeter added: clearance 0.2, trace_width 10, via_dia 0.8, via_drill 0.4
- net class Power added: clearance 0.2, trace_width 4, via_dia 0.8, via_drill 0.4
- net class Strom removed
- net class ower 5V added: clearance 0.2, trace_width 1, via_dia 0.8, via_drill 0.4
- board text added: "Fabian Heine Studienarbeit"

Commit message: Platine fertig
Parts:
- moved U3 1.93 mm to (176.7, 103.2)
- moved C10 0.43 mm to (163.6, 98.2)
- moved C11 0.40 mm to (163.6, 94.3)
Routing:
- net /Sheet5EE7EB52/-IN1: track 32.9 -> 20.7 mm, vias 0 -> 2
- net Net-(R11-Pad2): track 11.5 -> 9.35 mm
- net GND: track 27.4 -> 25.8 mm, vias 85 -> 176
- net /Sheet5EE7EB52/-IN2: track 41.2 -> 40.0 mm
- net +3V3: track 117.3 -> 118.2 mm
- net A3: track 24.9 -> 24.3 mm
- net /C13: track 4.79 -> 4.24 mm
- net MM4-: vias 1 -> 0
Other:
- board text added: "GND"
- board text added: "VBAT"
- board text added: "o"
